File: Schematics/ATDevBoard/ATDevBoard.sch (EAGLE design)
At the start: 40 parts, among them U1 TINY85-DIP

Commit message: Removed diode for reset line, revisted layout for oscillator
Parts:
- removed D4: 1N4007, diode:1N4004
- D2: value 1N4148 -> 1N4007; device adafruit:DIODESOD-323F -> diode:1N4004
Connections:
- net +3V3: now also D3.A; no longer D3.C, D4.A
- net N$1: now also D2.A; no longer D3.A
- net RESET: no longer D2.A
- net VIN: now also D3.C; no longer D4.C
Other:
- moved on the sheet: D3, R2
Changed lines of the file:
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@@
 <schematic xreflabel="%F%N/%S" xrefpart="/%S.%C%R">
 <attributes>
-<attribute name="VERSION" value="0.76"/>
+<attribute name="VERSION" value="0.77"/>
 </attributes>
 <variantdefs>
@@
 <part name="LM317T" library="v-reg" deviceset="LM317TS" device=""/>
 <part name="R1" library="rcl" deviceset="R-US_" device="0204/7" value="220"/>
+<part name="D2" library="diode" deviceset="1N4004" device="" value="1N4007"/>
 <part name="D3" library="diode" deviceset="1N4004" device="" value="1N4007"/>
-<part name="D4" library="diode" deviceset="1N4004" device="" value="1N4007"/>
 <part name="ICSP_10" library="SparkFun-Connectors" deviceset="AVR_SPI_PROG_5X2" device="PTH2" value="5x2 M"/>
 <part name="GND4" library="supply2" deviceset="GND" device=""/>
@@
 <part name="R5" library="rcl" deviceset="R-US_" device="0207/10" value="1K"/>
 <part name="R6" library="rcl" deviceset="R-US_" device="0207/10" value="1K"/>
-<part name="D2" library="adafruit" deviceset="DIODE" device="SOD-323F" value="1N4148"/>
 <part name="F1" library="SparkFun-Fuses" deviceset="PPTC" device="_PTH" value="90V/0.5A"/>
 <part name="SUPPLY2" library="supply2" deviceset="GND" device=""/>
@@
 </instance>
 <instance part="GND1" gate="GND" x="111.76" y="139.7"/>
-<instance part="P+2" gate="G$1" x="50.8" y="139.7" smashed="yes">
-<attribute name="VALUE" x="52.705" y="142.24" size="1.778" layer="96" rot="R180"/>
+<instance part="P+2" gate="G$1" x="50.8" y="157.48" smashed="yes">
+<attribute name="VALUE" x="52.705" y="160.02" size="1.778" layer="96" rot="R180"/>
 </instance>
 <instance part="P+3" gate="G$1" x="48.26" y="101.6" smashed="yes">
@@
 <instance part="AD" gate="A" x="152.4" y="106.68" rot="MR180"/>
 <instance part="GND5" gate="GND" x="33.02" y="139.7" rot="R90"/>
-<instance part="GND12" gate="GND" x="71.12" y="154.94"/>
+<instance part="GND12" gate="GND" x="66.04" y="154.94"/>
 <instance part="ON" gate="G$1" x="205.74" y="73.66" rot="MR90"/>
 <instance part="GND14" gate="GND" x="198.12" y="71.12" rot="MR0"/>
@@
 </instance>
 <instance part="C4" gate="G$1" x="124.46" y="152.4"/>
-<instance part="GND13" gate="GND" x="124.46" y="160.02" rot="R180"/>
+<instance part="GND13" gate="GND" x="132.08" y="152.4"/>
 <instance part="R7" gate="G$1" x="53.34" y="116.84" smashed="yes" rot="MR90">
 <attribute name="NAME" x="55.88" y="121.0564" size="1.778" layer="95" rot="MR180"/>
@@
 <instance part="LM317T" gate="1" x="241.3" y="162.56"/>
 <instance part="R1" gate="G$1" x="254" y="157.48" rot="R270"/>
-<instance part="D3" gate="1" x="248.92" y="157.48" rot="R90"/>
-<instance part="D4" gate="1" x="241.3" y="170.18" rot="R180"/>
+<instance part="D2" gate="1" x="248.92" y="157.48" rot="R90"/>
+<instance part="D3" gate="1" x="241.3" y="170.18" rot="R180"/>
 <instance part="ICSP_10" gate="G$1" x="93.98" y="170.18" smashed="yes">
 <attribute name="NAME" x="88.9" y="178.308" size="1.778" layer="95" font="vector"/>
@@
 </instance>
 <instance part="GND3" gate="GND" x="30.48" y="109.22" rot="MR0"/>
-<instance part="R2" gate="G$1" x="50.8" y="132.08" rot="R270"/>
+<instance part="R2" gate="G$1" x="50.8" y="149.86" rot="R270"/>
 <instance part="R3" gate="G$1" x="205.74" y="88.9" rot="MR0"/>
 <instance part="R4" gate="G$1" x="215.9" y="73.66"/>
 <instance part="R5" gate="G$1" x="264.16" y="83.82" rot="MR0"/>
 <instance part="R6" gate="G$1" x="264.16" y="73.66" rot="MR0"/>
-<instance part="D2" gate="G$1" x="58.42" y="132.08" smashed="yes" rot="R90">
-<attribute name="NAME" x="55.88" y="129.54" size="1.778" layer="95" rot="R90"/>
-<attribute name="VALUE" x="62.23" y="129.54" size="1.778" layer="96" rot="R90"/>
-</instance>
 <instance part="F1" gate="G$1" x="220.98" y="132.08"/>
 <instance part="SUPPLY2" gate="GND" x="213.36" y="119.38"/>
@@
 </segment>
 <segment>
-<wire x1="60.96" y1="157.48" x2="71.12" y2="157.48" width="0.1524" layer="91"/>
+<wire x1="60.96" y1="157.48" x2="66.04" y2="157.48" width="0.1524" layer="91"/>
 <wire x1="60.96" y1="157.48" x2="60.96" y2="154.94" width="0.1524" layer="91"/>
 <pinref part="GND12" gate="GND" pin="GND"/>
@@
 </segment>
 <segment>
-<wire x1="124.46" y1="157.48" x2="124.46" y2="154.94" width="0.1524" layer="91"/>
+<wire x1="132.08" y1="154.94" x2="124.46" y2="154.94" width="0.1524" layer="91"/>
 <pinref part="C4" gate="G$1" pin="1"/>
 <pinref part="GND13" gate="GND" pin="GND"/>
@@
 <pinref part="ICSP_10" gate="G$1" pin="RESET"/>
 <wire x1="86.36" y1="170.18" x2="76.2" y2="170.18" width="0.1524" layer="91"/>
-<wire x1="66.04" y1="124.46" x2="58.42" y2="124.46" width="0.1524" layer="91"/>
-<wire x1="58.42" y1="124.46" x2="50.8" y2="124.46" width="0.1524" layer="91"/>
-<wire x1="50.8" y1="124.46" x2="45.72" y2="124.46" width="0.1524" layer="91"/>
+<wire x1="66.04" y1="124.46" x2="45.72" y2="124.46" width="0.1524" layer="91"/>
 <wire x1="45.72" y1="142.24" x2="45.72" y2="137.16" width="0.1524" layer="91"/>
 <wire x1="45.72" y1="137.16" x2="45.72" y2="124.46" width="0.1524" layer="91"/>
-<wire x1="50.8" y1="127" x2="50.8" y2="124.46" width="0.1524" layer="91"/>
 <wire x1="86.36" y1="142.24" x2="76.2" y2="142.24" width="0.1524" layer="91"/>
 <wire x1="76.2" y1="142.24" x2="60.96" y2="142.24" width="0.1524" layer="91"/>
-<wire x1="60.96" y1="142.24" x2="45.72" y2="142.24" width="0.1524" layer="91"/>
+<wire x1="60.96" y1="142.24" x2="50.8" y2="142.24" width="0.1524" layer="91"/>
+<wire x1="50.8" y1="142.24" x2="45.72" y2="142.24" width="0.1524" layer="91"/>
 <wire x1="60.96" y1="144.78" x2="60.96" y2="142.24" width="0.1524" layer="91"/>
-<wire x1="58.42" y1="129.54" x2="58.42" y2="124.46" width="0.1524" layer="91"/>
-<junction x="50.8" y="124.46"/>
 <junction x="60.96" y="142.24"/>
-<junction x="58.42" y="124.46"/>
 <label x="55.88" y="125.095" size="1.778" layer="95"/>
 <label x="25.4" y="134.62" size="1.6764" layer="95"/>
@@
 <junction x="76.2" y="142.24"/>
 <pinref part="SW1" gate="G$1" pin="P$1"/>
-<pinref part="R2" gate="G$1" pin="2"/>
-<pinref part="D2" gate="G$1" pin="A"/>
 <pinref part="POWER" gate="A" pin="1"/>
 <wire x1="45.72" y1="137.16" x2="20.32" y2="137.16" width="0.1524" layer="91"/>
 <junction x="45.72" y="137.16"/>
+<pinref part="R2" gate="G$1" pin="2"/>
+<wire x1="50.8" y1="144.78" x2="50.8" y2="142.24" width="0.1524" layer="91"/>
+<junction x="50.8" y="142.24"/>
 </segment>
 <segment>
@@
 <wire x1="228.6" y1="162.56" x2="233.68" y2="162.56" width="0.1524" layer="91"/>
 <junction x="228.6" y="162.56"/>
-<pinref part="D4" gate="1" pin="C"/>
+<pinref part="D3" gate="1" pin="C"/>
 <wire x1="238.76" y1="170.18" x2="228.6" y2="170.18" width="0.1524" layer="91"/>
 <wire x1="228.6" y1="170.18" x2="228.6" y2="162.56" width="0.1524" layer="91"/>
@@
 </segment>
 <segment>
-<wire x1="50.8" y1="137.16" x2="58.42" y2="137.16" width="0.1524" layer="91"/>
-<wire x1="58.42" y1="137.16" x2="58.42" y2="134.62" width="0.1524" layer="91"/>
 <pinref part="P+2" gate="G$1" pin="+3V3"/>
 <pinref part="R2" gate="G$1" pin="1"/>
-<junction x="50.8" y="137.16"/>
-<pinref part="D2" gate="G$1" pin="C"/>
 </segment>
 <segment>
@@
 <wire x1="254" y1="162.56" x2="266.7" y2="162.56" width="0.1524" layer="91"/>
 <junction x="254" y="162.56"/>
-<pinref part="D4" gate="1" pin="A"/>
+<pinref part="D3" gate="1" pin="A"/>
 <wire x1="243.84" y1="170.18" x2="254" y2="170.18" width="0.1524" layer="91"/>
 <wire x1="254" y1="170.18" x2="254" y2="162.56" width="0.1524" layer="91"/>
-<pinref part="D3" gate="1" pin="C"/>
+<pinref part="D2" gate="1" pin="C"/>
 <wire x1="248.92" y1="160.02" x2="248.92" y2="162.56" width="0.1524" layer="91"/>
 <junction x="248.92" y="162.56"/>
@@
 <pinref part="LM317T" gate="1" pin="ADJ"/>
 <wire x1="248.92" y1="149.86" x2="241.3" y2="149.86" width="0.1524" layer="91"/>
-<pinref part="D3" gate="1" pin="A"/>
+<pinref part="D2" gate="1" pin="A"/>
 <wire x1="248.92" y1="154.94" x2="248.92" y2="149.86" width="0.1524" layer="91"/>
 <junction x="248.92" y="149.86"/>

Commit message: Replaced USB micro connector with Molex one
Parts:
- R8: value (none) -> 2K
- USB1: value ZX62-B-5PA -> MOLEX47589; device Seeed-Connector:MICRO-USB-SMD(ZX62-B-5PA) -> con-molex-usb:MICRO-USB-RECEPTACLE47589-0001
Connections:
- removed net VBUS: F1.1, USB1.VBUS
- new net VUSB: F1.1, USB1.1
- net GND: now also USB1.5; no longer USB1.GND
Other:
- moved on the sheet: F1
Changed lines of the file:
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@@
 </class>
 <class number="2" name="gnd" width="0.4064" drill="0.508">
-<clearance class="2" value="0.254"/>
+<clearance class="2" value="0.127"/>
 </class>
 <class number="3" name="aref" width="0.4064" drill="0.508">
@@
 <part name="F1" library="SparkFun-Fuses" deviceset="PPTC" device="_PTH" value="90V/0.5A"/>
 <part name="SUPPLY2" library="supply2" deviceset="GND" device=""/>
-<part name="USB1" library="Seeed-Connector" deviceset="MICRO-USB-SMD(ZX62-B-5PA)" device="" value="ZX62-B-5PA"/>
-<part name="R8" library="bourns" deviceset="3362" device="R"/>
+<part name="R8" library="bourns" deviceset="3362" device="R" value="2K"/>
+<part name="USB1" library="con-molex-usb" deviceset="MICRO-USB-RECEPTACLE" device="47589-0001" value="MOLEX47589"/>
 </parts>
 <sheets>
@@
 <instance part="R5" gate="G$1" x="264.16" y="83.82" rot="MR0"/>
 <instance part="R6" gate="G$1" x="264.16" y="73.66" rot="MR0"/>
-<instance part="F1" gate="G$1" x="220.98" y="132.08"/>
-<instance part="SUPPLY2" gate="GND" x="213.36" y="119.38"/>
-<instance part="USB1" gate="G$1" x="198.12" y="121.92"/>
+<instance part="F1" gate="G$1" x="213.36" y="134.62"/>
+<instance part="SUPPLY2" gate="GND" x="203.2" y="121.92"/>
 <instance part="R8" gate="G$1" x="241.3" y="144.78"/>
+<instance part="USB1" gate="G$1" x="195.58" y="129.54" rot="MR0"/>
 </instances>
 <busses>
@@
 </segment>
 <segment>
-<pinref part="SUPPLY2" gate="GND" pin="GND"/>
-<pinref part="USB1" gate="G$1" pin="GND"/>
-<wire x1="213.36" y1="121.92" x2="208.28" y2="121.92" width="0.1524" layer="91"/>
-</segment>
-<segment>
 <pinref part="GND5" gate="GND" pin="GND"/>
 <pinref part="POWER" gate="A" pin="2"/>
@@
 <wire x1="27.94" y1="142.24" x2="27.94" y2="139.7" width="0.1524" layer="91"/>
 <junction x="27.94" y="139.7"/>
+</segment>
+<segment>
+<pinref part="USB1" gate="G$1" pin="5"/>
+<pinref part="SUPPLY2" gate="GND" pin="GND"/>
+<wire x1="200.66" y1="124.46" x2="203.2" y2="124.46" width="0.1524" layer="91"/>
 </segment>
 </net>
@@
 <junction x="215.9" y="162.56"/>
 <pinref part="F1" gate="G$1" pin="2"/>
-<wire x1="228.6" y1="132.08" x2="233.68" y2="132.08" width="0.1524" layer="91"/>
-<wire x1="233.68" y1="132.08" x2="233.68" y2="162.56" width="0.1524" layer="91"/>
+<wire x1="220.98" y1="134.62" x2="233.68" y2="134.62" width="0.1524" layer="91"/>
+<wire x1="233.68" y1="134.62" x2="233.68" y2="162.56" width="0.1524" layer="91"/>
 <junction x="233.68" y="162.56"/>
 <label x="220.98" y="162.56" size="1.778" layer="95" font="vector"/>
@@
 </segment>
 </net>
-<net name="VBUS" class="4">
+<net name="VUSB" class="0">
 <segment>
 <pinref part="F1" gate="G$1" pin="1"/>
-<wire x1="215.9" y1="132.08" x2="213.36" y2="132.08" width="0.1524" layer="91"/>
-<pinref part="USB1" gate="G$1" pin="VBUS"/>
-<wire x1="213.36" y1="132.08" x2="212.09" y2="132.08" width="0.1524" layer="91"/>
-<wire x1="212.09" y1="132.08" x2="208.28" y2="132.08" width="0.1524" layer="91"/>
-</segment>
-</net>
+<pinref part="USB1" gate="G$1" pin="1"/>
+<wire x1="208.28" y1="134.62" x2="200.66" y2="134.62" width="0.1524" layer="91"/>
+<label x="200.66" y="132.08" size="1.778" layer="95" font="vector"/>
+</segment>
+</net>

Commit message: Fidex schematic for trimmer, added jumper for VCC, schematic tested on breadboard
Parts:
- removed C5: 100uf, SparkFun-Capacitors:CAP_POLPTH1
- added JP1: (no value), jumper:JP1E
- ON: value GREEN -> RED
Connections:
- removed net +3V3: C1.2, C2.2, C6.2, C9.2, D2.C, D3.A, ICSP_10.VCC, ICSP_6.2, LM317T.OUT, MCU1.VCC, POWER.4, R1.1, R2.1, R4.2, R5.1, R6.1, U1.VCC, ZU4.AVCC, ZU4.VCC
- new net N$5: D2.C, D3.A, JP1.1, LM317T.OUT, R1.1
- new net VCC: C1.2, C2.2, C6.2, C9.2, ICSP_10.VCC, ICSP_6.2, JP1.2, MCU1.VCC, POWER.4, R2.1, R4.2, R5.1, R6.1, U1.VCC, ZU4.AVCC, ZU4.VCC
- net GND: no longer C5.-
- net N$1: now also R8.2; no longer R8.3
- net VIN: no longer C5.+
Other:
- moved on the sheet: C8, C9, D1, D2, D3, F1, JPOWER, LM317T, R1, R8, USB1

Commit message: Modified cutout slots for DC connector and micro USB, reviewed name texts in tNames level. Made gerber file for board v1.0, ready for SeeedStudio
Parts:
- USB1: device con-molex-usb:MICRO-USB-RECEPTACLE47589-0001 -> CuSTOM_GB:MICRO-USB-RECEPTACLE47589-0001
- renumbered R8 to TRIM1
Other:
- note added: "Atmel development board, with support for ATMega328p, ATTinyX4, ATTinyX5."
- note added: "License: Apache v2.0"
Changed lines of the file:
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@@
 <schematic xreflabel="%F%N/%S" xrefpart="/%S.%C%R">
 <attributes>
-<attribute name="VERSION" value="0.78"/>
+<attribute name="VERSION" value="1.0"/>
 </attributes>
 <variantdefs>
@@
 <part name="F1" library="SparkFun-Fuses" deviceset="PPTC" device="_PTH" value="90V/0.5A"/>
 <part name="SUPPLY2" library="supply2" deviceset="GND" device=""/>
-<part name="R8" library="bourns" deviceset="3362" device="R" value="2K"/>
-<part name="USB1" library="con-molex-usb" deviceset="MICRO-USB-RECEPTACLE" device="47589-0001" value="MOLEX47589"/>
+<part name="TRIM1" library="bourns" deviceset="3362" device="R" value="2K"/>
+<part name="USB1" library="CuSTOM_GB" deviceset="MICRO-USB-RECEPTACLE" device="47589-0001" value="MOLEX47589"/>
 <part name="JP1" library="jumper" deviceset="JP1E" device=""/>
 <part name="P+9" library="supply1" deviceset="VCC" device=""/>
@@
 <text x="154.94" y="101.6" size="1.778" layer="91">RX X4</text>
 <text x="154.94" y="99.06" size="1.778" layer="91">TX X4</text>
+<text x="187.96" y="33.02" size="1.778" layer="97">Atmel development board, with support
+for ATMega328p, ATTinyX4, ATTinyX5.</text>
+<text x="254" y="33.02" size="1.778" layer="91">License: Apache v2.0</text>
 </plain>
 <instances>
@@
 <instance part="F1" gate="G$1" x="220.98" y="132.08"/>
 <instance part="SUPPLY2" gate="GND" x="210.82" y="119.38"/>
-<instance part="R8" gate="G$1" x="246.38" y="139.7"/>
+<instance part="TRIM1" gate="G$1" x="246.38" y="139.7"/>
 <instance part="USB1" gate="G$1" x="203.2" y="127" rot="MR0"/>
 <instance part="JP1" gate="A" x="264.16" y="162.56"/>
@@
 </segment>
 <segment>
-<pinref part="R8" gate="G$1" pin="1"/>
+<pinref part="TRIM1" gate="G$1" pin="1"/>
 <pinref part="SUPPLY1" gate="GND" pin="GND"/>
 <wire x1="246.38" y1="134.62" x2="246.38" y2="132.08" width="0.1524" layer="91"/>
@@
 <pinref part="D2" gate="1" pin="A"/>
 <wire x1="251.46" y1="152.4" x2="251.46" y2="147.32" width="0.1524" layer="91"/>
-<pinref part="R8" gate="G$1" pin="2"/>
+<pinref part="TRIM1" gate="G$1" pin="2"/>
 <wire x1="251.46" y1="147.32" x2="251.46" y2="139.7" width="0.1524" layer="91"/>
 <junction x="251.46" y="147.32"/>
